File: 0009_Touch_Module_ESP32_PIN.kicad_sch (KiCad schematic)
At the start: 12 parts

Commit message: Add files via upload
Parts:
- removed C4, C5, C6: 0.1uF, symbol Device:C_Small
- added D4: LED, LED_SMD:LED_0603_1608Metric, symbol Device:LED
- added R1: 470R, Resistor_SMD:R_0603_1608Metric, symbol Device:R
- added U4: ~, Moduler_:pin_header, symbol moduler_pin:air
- C1, C2, C3: footprint (none) -> Capacitor_SMD:C_0603_1608Metric
- U1, U2, U3: footprint (none) -> Library:touch
Connections:
- net DIN2 is gone; now on an unnamed net: D2.4 (DIN)
- net DIN3 is gone; now on an unnamed net: D3.4 (DIN)
- net +5V: now also R1.1, U4.7
- net GND: now also D4.1 (K), U4.9
- net TOUCH1: now also U1.1, U4.12; no longer U1.touch
- net TOUCH2: now also U2.1, U4.13; no longer U2.touch
- net TOUCH3: now also U3.1, U4.14; no longer U3.touch
- net DOUT: now reaches D3.2 (DOUT)
- net DOUT: now also U4.16
- net DIN1 renamed DIN
- net DIN: now also U4.15
- new net: D4.2 (A), R1.2
- no-connect marks 0 -> 11
Other:
- moved on the sheet: C1, C2, C3, D1, D2, D3, U1, U2, U3
